File: Hardware/Project/CPU.sch (KiCad schematic (older format))
At the start: 25 parts, among them SW1 SW_Push, U1 STC89C52, U11 74LS00, U2 74LS373, U3 74LS00, U4 28C256, U5 74LS138, U7 74LS133, Y1 Crystal

Commit message: 1
Parts:
- removed Q?: 2N3906, Package_TO_SOT_THT:TO-92_Inline, symbol Transistor_BJT:2N3906
- removed R? (x9): 1k, Resistor_SMD:R_0805_2012Metric, symbol Device:R
- removed U11: 74LS00, symbol 74xx:74LS00
- removed unit 5 of U3
- removed U5: 74LS138, symbol 74xx:74LS138
- removed U7: 74LS133, symbol 74xx:74LS133
- added R3, R4, R5, R6: 1k, Resistor_SMD:R_0805_2012Metric, symbol Device:R
- added U11: 74LS30, symbol 74xx:74LS30
- added U13, U7: 74LS32, symbol 74xx:74LS32
- added U?: 74LS00, symbol 74xx:74LS00
- U1: symbol Vintage:STC89C52 -> 8051-rescue:STC89C52-Vintage
Connections:
- net labels added: ISP, MEM_ERR, ~IORQ, ~ISP, ~MEMRQ, ~RD0, ~WR0
- net labels removed: ~A15, ~BIOS_CS, ~IO0_CS, ~IO1_CS, ~IO2_CS, ~IO3_CS, ~IO4_CS, ~IO5_CS, ~IO6_CS, ~IO7_CS, ~IO_CS, ~RAM_CS
- wire segments 267 -> 232
Other:
- note added: "IO ADDRESS = 1111 1111 0xxx xxxx (FF00-FF7F) \n////////////////////////////////////////////////////////////////////////////////////\n/ISP /BOOTING /WR /RD | /WR0 /RD0 /WR1 /RD1\n0 0 0 0 | x x x x // NOT POSSIBLE\n0 0 0 1 | x x x x // NOT POSSIBLE\n0 0 1 0 | x x x x\n0 0 1 1 | x x x x // NOT POSSIBLE\n\n0 1 0 0 | x x x x // NOT POSSIBLE\n0 1 0 1 | 0 1 1 1 // ISP\n0 1 1 0 | 1 1 1 0\n0 1 1 1 | 1 1 1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"
- note removed: "IO ADDRESS = 1111 1111 0xxx xxxx (FF00-FF7F) \n\n/BOOTING A15 /IO_CS | /BIOS_CS /RAM_CS\n0 0 0 | 0 1\n0 0 1 | 0 1\n0 1 0 | 1 1\n0 1 1 | 1 0\n1 0 0 | 1 1\n1 0 1 | 1 0\n1 1 0 | 1 1 \n1 1 1 | 1 0\n\n/IO_CS = /(A15 * A14 * A13 * A12 * A11 * A10 * A9 * A8 * A7')\n/BIOS_CS = /BOOTING + A15 = (/BOOTING' * A15')' = (BOOTING * /A15)'\n/RAM_CS = /BOOTING' * A15' + /IO_CS' = ( ((BOOTING * A15')') * (/IO_CS)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"
- moved on the sheet: C1, C2, C3, C4, R1, R2, SW1, U2, U3A, U3B, U3C, U4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

Commit message: 1
Parts:
- removed R2, R3, R4, R5, R6: 1k, Resistor_SMD:R_0805_2012Metric, symbol Device:R
- removed U11: 74LS30, symbol 74xx:74LS30
- removed U13, U7: 74LS32, symbol 74xx:74LS32
- removed U4: 28C256, symbol Memory_EEPROM:28C256
- removed U?: 74LS00, symbol 74xx:74LS00
- added D?: DIODE, symbol pspice:DIODE
- added RN1: R_Network08, Resistor_THT:R_Array_SIP9, symbol Device:R_Network08
- added U11, U8: 74LS32, symbol 74xx:74LS32
- added U14: 28C256, symbol Memory_EEPROM:28C256
- added unit 4 of U3
- added U4: 74LS14, symbol 74xx:74LS14
- added U5, U7: 74LS138, symbol 74xx:74LS138
- added U9: 74LS30, symbol 74xx:74LS30
Connections:
- net labels added: ~ENTER_ISP, ~IO0_CS, ~IO1_CS, ~IO2_CS, ~IO3_CS, ~IO4_CS, ~IO5_CS, ~IO6_CS, ~IO7_CS, ~IOREQ, ~RESET, ~WARM_BOOT
- net labels removed: MEM_ERR, RESET
- wire segments 232 -> 280
Other:
- note added: "1111 1111 0111 xxxx (FF70-FF7F)\nFF70 = ~EXIT_BOOT\nFF71 = ~ENTER_ISP\nFF72\nFF73\nFF74\nFF75\nFF76\nFF77"
- note added: "1111 1111 0xxx xxxx (FF00-FF7F) \n~IO0_CS~ = (FF00-FF0F)\n~IO1_CS~ = (FF10-FF1F)\n~IO2_CS~ = (FF20-FF2F)\n~IO3_CS~ = (FF30-FF3F)\n~IO4_CS~ = (FF40-FF4F)\n~IO5_CS~ = (FF50-FF5F)\n~IO6_CS~ = (FF60-FF6F)\n~IO7_CS~ = (FF70-FF7F)"
- note added: "IO ADDRESS = 1111 1111 0xxx xxxx (FF00-FF7F) \n\n///////////////////////////////////////////////////////\n/ISP /BOOTING /WR /RD | /WR0 /RD0 /WR1 /RD1\n0 0 0 0 | x x x x // NOT POSSIBLE\n0 0 0 1 | x x x x // NOT POSSIBLE\n0 0 1 0 | x x x x\n0 0 1 1 | x x x x // NOT POSSIBLE\n\n0 1 0 0 | x x x x // NOT POSSIBLE\n0 1 0 1 | 0 1 1 1 // ISP\n0 1 1 0 | 1 1 1 0\n0 1 1 1 | 1 1 1 1\n\n1 0 0 0 | x x x x // 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"
- note removed: "IO ADDRESS = 1111 1111 0xxx xxxx (FF00-FF7F) \n////////////////////////////////////////////////////////////////////////////////////\n/ISP /BOOTING /WR /RD | /WR0 /RD0 /WR1 /RD1\n0 0 0 0 | x x x x // NOT POSSIBLE\n0 0 0 1 | x x x x // NOT POSSIBLE\n0 0 1 0 | x x x x\n0 0 1 1 | x x x x // NOT POSSIBLE\n\n0 1 0 0 | x x x x // NOT POSSIBLE\n0 1 0 1 | 0 1 1 1 // ISP\n0 1 1 0 | 1 1 1 0\n0 1 1 1 | 1 1 1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"
- moved on the sheet: C1, C2, C3, C4, R1, SW1, U1, U2, U3A, U3B, Y1

Commit message: 1
Parts:
- added Q1: Q_PNP_CBE, symbol Device:Q_PNP_CBE
- added R2, R3, R4: 1k, Resistor_SMD:R_0805_2012Metric, symbol Device:R
- U1: symbol 8051-rescue:STC89C52-Vintage -> 8051-rescue:STC89C52-Vintage-8051-rescue
- gave numbers to parts that had none: 1
Connections:
- net labels added: RESET, ~CPU_RD, ~CPU_WR, ~RD_BIOS, ~WR_BIOS
- net labels removed: ~IOREQ, ~RD0, ~WR0
- wire segments 280 -> 297
Other:
- note added: "1111 1111 0111 xxxx (FF70-FF7F)\nFF70 = ~EXIT_BOOT\nFF71 = ~ENTER_ISP\nFF72 = ~WARM_BOOT\nFF73\nFF74\nFF75\nFF76\nFF77"
- note removed: "1111 1111 0111 xxxx (FF70-FF7F)\nFF70 = ~EXIT_BOOT\nFF71 = ~ENTER_ISP\nFF72\nFF73\nFF74\nFF75\nFF76\nFF77"
- moved on the sheet: C1, D1, R1, SW1, U4A

Commit message: 123
Parts:
- removed U14: 28C256, symbol Memory_EEPROM:28C256
- removed unit 1 of U4
- added C4: C, Capacitor_SMD:C_0805_2012Metric, symbol Device:C
- added R11: 1k, Resistor_SMD:R_0805_2012Metric, symbol Device:R
- added R7: 1M, Resistor_SMD:R_0805_2012Metric, symbol Device:R
- added U12: 74LS08, Package_DIP:DIP-14_W7.62mm_Socket, symbol 74xx:74LS08
- added unit 5 of U13
- added unit 5 of U15
- added unit 2 of U18
- added unit 5 of U19
- added unit 7 of U9
- added unit 3 of U9
- added unit 4 of U9
- added unit 5 of U9
- added Y1: Crystal, Connector_PinSocket_2.54mm:PinSocket_1x02_P2.54mm_Vertical, symbol Device:Crystal
- D2: renamed from D1; footprint (none) -> LED_SMD:LED_0805_2012Metric
- Q1: footprint (none) -> Button_Switch_Keyboard:SW_Cherry_MX1A_1.00u_PCB
- SW1: footprint (none) -> Connector_PinSocket_2.54mm:PinSocket_1x02_P2.54mm_Vertical
- U11: renamed from U7; footprint (none) -> Package_DIP:DIP-18_W7.62mm_Socket
- U13: renamed from U3; footprint (none) -> Package_DIP:DIP-14_W7.62mm_Socket
- U14: renamed from U1; footprint (none) -> Package_DIP:DIP-40_W25.4mm_Socket; symbol 8051-rescue:STC89C52-Vintage-8051-rescue -> 8051-rescue:STC89C52-Vintage-8051-rescue-8051-rescue
- U15: renamed from U8; footprint (none) -> Package_DIP:DIP-14_W7.62mm_Socket
- U16: renamed from U2; footprint (none) -> Package_DIP:DIP-20_W7.62mm_Socket
- U18: renamed from U9; footprint (none) -> Package_DIP:DIP-14_W7.62mm_Socket
- U19: renamed from U11; footprint (none) -> Package_DIP:DIP-14_W7.62mm_Socket
- U20: renamed from U5; footprint (none) -> Package_DIP:DIP-16_W7.62mm_Socket
- U9: renamed from U4; footprint (none) -> Package_DIP:DIP-14_W7.62mm_Socket
- Y2: renamed from Y1; footprint (none) -> Connector_PinSocket_2.54mm:PinSocket_1x02_P2.54mm_Vertical
- renumbered C1 to C3, C3 to C5, C4 to C6, R4 to R10, R2 to R6, R3 to R8, R1 to R9
Connections:
- net labels added: ~PSEN
- wire segments 297 -> 314
Other:
- moved on the sheet: C3, C5, C6, D2, Q1, R6, R9, RN1, SW1, U14, U15A, U15B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
