File: Hardware/Project/CPU.sch (KiCad schematic (older format))
At the start: 27 parts, among them Q1 Q_PNP_CBE, SW1 SW_Push, U11 74LS138, U12 74LS08, U13 74LS00, U14 STC89C52, U15 74LS32, U16 74LS373, U18 74LS30, U19 74LS32, U20 74LS138, U9 74LS14, Y1 Crystal, Y2 Crystal

Commit message: 1
Parts:
- Q1: footprint Button_Switch_Keyboard:SW_Cherry_MX1A_1.00u_PCB -> Package_TO_SOT_THT:TO-92
Changed lines of the file:
@@
 F 0 "Q1" H 3191 4546 50  0000 L CNN
 F 1 "Q_PNP_CBE" H 3191 4455 50  0000 L CNN
-F 2 "Button_Switch_Keyboard:SW_Cherry_MX1A_1.00u_PCB" H 3200 4600 50  0001 C CNN
+F 2 "Package_TO_SOT_THT:TO-92" H 3200 4600 50  0001 C CNN
 F 3 "~" H 3000 4500 50  0001 C CNN
 	1    3000 4500

Commit message: 1
Parts:
- removed C2, C4: C, Capacitor_SMD:C_0805_2012Metric, symbol Device:C
- removed R11: 1k, Resistor_SMD:R_0805_2012Metric, symbol Device:R
- removed R7: 1M, Resistor_SMD:R_0805_2012Metric, symbol Device:R
- removed U14: STC89C52, Package_DIP:DIP-40_W25.4mm_Socket, symbol 8051-rescue:STC89C52-Vintage-8051-rescue-8051-rescue
- removed U16: 74LS373, Package_DIP:DIP-20_W7.62mm_Socket, symbol 74xx:74LS373
- removed unit 3 of U9
- removed unit 4 of U9
- removed unit 5 of U9
- removed unit 2 of U9
- removed Y1: Crystal, Connector_PinSocket_2.54mm:PinSocket_1x02_P2.54mm_Vertical, symbol Device:Crystal
- added C1: CP1, Capacitor_THT:CP_Radial_D7.5mm_P2.50mm, symbol Device:CP1
- added D2: ~BOOTING, LED_SMD:LED_0805_2012Metric, symbol Device:LED
- added D3: ~ISP, LED_SMD:LED_0805_2012Metric, symbol Device:LED
- added D4: POWER, LED_SMD:LED_0805_2012Metric, symbol Device:LED
- added J1: USB_B_Mini, Connector_USB:USB_Micro-B_Wuerth_629105150521_CircularHoles, symbol Connector:USB_B_Mini
- added J2: Conn_02x20_Odd_Even, Connector_PinHeader_2.54mm:PinHeader_2x20_P2.54mm_Vertical, symbol Connector_Generic:Conn_02x20_Odd_Even
- added R13, R14, R15: 330, Resistor_SMD:R_0805_2012Metric, symbol Device:R
- added R3: 1k, Resistor_SMD:R_0805_2012Metric, symbol Device:R
- added unit 1 of U11
- added unit 2 of U11
- added U13: STC89C52-Vintage, Package_DIP:DIP-40_W15.24mm_Socket, symbol 8051-rescue:STC89C52-Vintage
- added U2: 74LS373_ARRANGED, Package_DIP:DIP-20_W7.62mm_Socket, symbol 8051-rescue:74LS373_ARRANGED
- added U20: AT29C512, Package_DIP:DIP-32_W15.24mm_Socket, symbol 8051-rescue:AT29C512
- C2: renamed from C3; footprint Capacitor_THT:CP_Radial_D4.0mm_P1.50mm -> Capacitor_THT:CP_Radial_D7.5mm_P2.50mm
- Q1: value Q_PNP_CBE -> 9015
- SW1: value SW_Push -> reset; footprint Connector_PinSocket_2.54mm:PinSocket_1x02_P2.54mm_Vertical -> Button_Switch_THT:SW_PUSH_6mm
- U10: renamed from U11; footprint Package_DIP:DIP-18_W7.62mm_Socket -> Package_DIP:DIP-16_W7.62mm_Socket
- Y2: footprint Connector_PinSocket_2.54mm:PinSocket_1x02_P2.54mm_Vertical -> Crystal:Crystal_HC18-U_Vertical
- renumbered C5 to C3, C6 to C4, D2 to D1, R6 to R1, R8 to R10, R10 to R11, R9 to R2, U9 to U11, U13 to U12, U12 to U14, U15 to U18, U18 to U19, U19 to U21, U20 to U22
Connections:
- net labels removed: ~PSEN
- wire segments 314 -> 384
Other:
- moved on the sheet: C3, C4, R10, R11, RN1, U10, U11G, U12A, U12B, U12C, U12D, U12E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

Commit message: 1
Parts:
- added C10, C12, C13, C14, C15, C16, C17, C18, C19, C20, C22: 1uf, Capacitor_SMD:C_0805_2012Metric, symbol Device:C
- added C11: C, Capacitor_SMD:C_0805_2012Metric, symbol Device:C
- added C21: CP1, Capacitor_THT:CP_Radial_D7.5mm_P2.50mm, symbol Device:CP1
- added R12, R16, R8, R9: 2k, Resistor_SMD:R_0805_2012Metric, symbol Device:R
- added R4, R5, R6, R7: 120, Resistor_SMD:R_0805_2012Metric, symbol Device:R
- added SW2: SW_DPDT_x2, Package_DIP:DIP-6_W7.62mm, symbol Switch:SW_DPDT_x2
- added U3: PS2_DUAL, Connector_PinSocket_2.54mm:PS2DUAL, symbol VGMPlayer-rescue:PS2_DUAL
Connections:
- net labels added: KEYBOARD_CLK, KEYBOARD_DAT, MOUSE_CLK, MOUSE_DAT
- wire segments 384 -> 492
Other:
- note added: "http://www.eeworld.com.cn/mcu/article_2017122636961.html\n"
- moved on the sheet: C1, J1, R2

Commit message: 1
Parts:
- U3: symbol VGMPlayer-rescue:PS2_DUAL -> 8051-rescue:PS2_DUAL-VGMPlayer-rescue
Connections:
- net labels removed: ~R, ~S
- wire segments 492 -> 491
Other:
- moved on the sheet: D2, D3, D4, R11, R13, R14, R15, U12A, U12B, U12C, U12D, U18A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

Commit message: 1
Parts:
- added C?: 0.05uF, Capacitor_SMD:C_0805_2012Metric, symbol Device:C
- added R? (x4): 10k, Resistor_SMD:R_0805_2012Metric, symbol Device:R
- added R? (x2): 1k, Resistor_SMD:R_0805_2012Metric, symbol Device:R
- added R?: 1.5k, Resistor_SMD:R_0805_2012Metric, symbol Device:R
- added R?: 3k, Resistor_SMD:R_0805_2012Metric, symbol Device:R
- added R?: 15k, Resistor_SMD:R_0805_2012Metric, symbol Device:R
- added unit 4 of U11
- added unit 5 of U11
- added unit 6 of U11
- added U?: Z80CPU, symbol CPU:Z80CPU
- added U?: 65C02, symbol 8051-rescue:65C02
- added U? (x4): 74LS14, Package_DIP:DIP-14_W7.62mm_Socket, symbol 74xx:74LS14
- added Y?: 2MHz, Crystal:Crystal_HC18-U_Vertical, symbol Device:Crystal
- added Y?: 4MHz, Crystal:Crystal_HC18-U_Vertical, symbol Device:Crystal
- J1: footprint Connector_USB:USB_Micro-B_Wuerth_629105150521_CircularHoles -> Connector_USB:USB_A_CNCTech_1001-011-01101_Horizontal
Connections:
- net A0: now also U?.30 (A0), U?.9 (A0)
- net A1: now also U?.10 (A1), U?.31 (A1)
- net A10: now also U?.19 (A10), U?.40 (A10)
- net A11: now also U?.1 (A11), U?.20 (A11)
- net A12: now also U?.2 (A12), U?.22 (A12)
- net A13: now also U?.23 (A13), U?.3 (A13)
- net A14: now also U?.24 (A14), U?.4 (A14)
- net A15: now also U?.25 (A15), U?.5 (A15)
- net A2: now also U?.11 (A2), U?.32 (A2)
- net A3: now also U?.12 (A3), U?.33 (A3)
- net A4: now also U?.13 (A4), U?.34 (A4)
- net A5: now also U?.14 (A5), U?.35 (A5)
- net A6: now also U?.15 (A6), U?.36 (A6)
- net A7: now also U?.16 (A7), U?.37 (A7)
- net A8: now also U?.17 (A8), U?.38 (A8)
- net A9: now also U?.18 (A9), U?.39 (A9)
- net D0: now also U?.14 (D0), U?.33 (D0)
- net D1: now also U?.15 (D1), U?.32 (D1)
- net D2: now also U?.12 (D2), U?.31 (D2)
- net D3: now also U?.30 (D3), U?.8 (D3)
- net D4: now also U?.29 (D4), U?.7 (D4)
- net D5: now also U?.28 (D5), U?.9 (D5)
- net D6: now also U?.10 (D6), U?.27 (D6)
- net D7: now also U?.13 (D7), U?.26 (D7)
- net ~CPU_RD: now also U?.21 (~RD~), U?.6
- net ~CPU_WR: now also U?.22 (~WR~), U?.34 (R/~W), U?.5
- net ~RESET: now also U?.26 (~RESET~), U?.40 (~RESET~)
- new net: R?.1, R?.1, R?.1, R?.1, U?.11 (VCC)
- new net: R?.2, U?.16 (~INT~), U?.4 (~IRQ~)
- new net: R?.2, U?.17 (~NMI~), U?.6 (~NMI~)
- new net: R?.2, U?.2 (RDY), U?.24 (~WAIT~)
- new net: R?.2, U?.25 (~BUSRQ~)
- new net: U11.12, U?.37 (Phi0(In)), U?.6 (~CLK~)
- new net: C?.1, R?.2, U11.8
- new net: R?.1, U11.9, Y?.2
- new net: R?.1, U11.10, U11.13, Y?.1
- new net: C?.2, R?.2, U11.11
- new net: U?.1 (VSS), U?.21 (VSS), U?.8 (VSS)
- new net: R?.1, R?.2, U?.11, U?.8
- new net: R?.1, R?.2, U?.9, Y?.2
- new net: R?.2, U?.10, U?.13, Y?.1
