File: Hardware/Project/8051.sch (KiCad schematic (older format))
At the start: 0 parts

Commit message: 1
Changed lines of the file:
@@
 EESchema Schematic File Version 4
+LIBS:8051-cache
 EELAYER 26 0
 EELAYER END
 $Descr A4 11693 8268
 encoding utf-8
-Sheet 1 5
+Sheet 1 6
 Title ""
 Date ""
@@
 F28 "D6" I R 3800 3450 50
 F29 "D7" I R 3800 3550 50
-F30 "~IO0_CS" I R 3800 4000 50
-F31 "~IO1_CS" I R 3800 4100 50
-F32 "~IO2_CS" I R 3800 4200 50
-F33 "~IO3_CS" I R 3800 4300 50
-F34 "~IO4_CS" I R 3800 4400 50
-F35 "~IO5_CS" I R 3800 4500 50
-F36 "~IO6_CS" I R 3800 4600 50
-F37 "~IO7_CS" I R 3800 4700 50
-F38 "~RAM_CS" I R 3800 4850 50
-F39 "RESET" I R 3800 5150 50
+F30 "RESET" I R 3800 5150 50
+F31 "~IORQ" I R 3800 3900 50
+F32 "~MEMRQ" I R 3800 4000 50
 $EndSheet
 $Sheet
@@
 F2 "A0" I R 4750 1250 50
 F3 "A1" I R 4750 1350 50
-F4 "A2" I R 4750 1450 50
-F5 "A3" I R 4750 1550 50
 F6 "A4" I R 4750 1650 50
 F7 "A5" I R 4750 1750 50
 F8 "A6" I R 4750 1850 50
-F9 "A7" I R 4750 1950 50
-F10 "A8" I R 4750 2050 50
-F11 "A9" I R 4750 2150 50
-F12 "A10" I R 4750 2250 50
-F13 "A11" I R 4750 2350 50
-F14 "A12" I R 4750 2450 50
-F15 "A13" I R 4750 2550 50
-F16 "A14" I R 4750 2650 50
-F17 "A15" I R 4750 2750 50
 F18 "~WR" I R 4750 3800 50
 F19 "~RD" I R 4750 3700 50
@@
 F28 "D6" I R 4750 3450 50
 F29 "D7" I R 4750 3550 50
-F30 "~IO0_CS" I R 4750 4000 50
-F31 "~IO1_CS" I R 4750 4100 50
-F32 "~IO2_CS" I R 4750 4200 50
-F33 "~IO3_CS" I R 4750 4300 50
-F34 "~IO4_CS" I R 4750 4400 50
-F35 "~IO5_CS" I R 4750 4500 50
-F36 "~IO6_CS" I R 4750 4600 50
-F37 "~IO7_CS" I R 4750 4700 50
-F38 "RESET" I R 4750 5150 50
+F30 "RESET" I R 4750 5150 50
+F31 "~IOREQ" I R 4750 3900 50
 $EndSheet
 $Sheet
-S 5000 1050 750  4300
-U 5E02D9A0
+S 4950 1050 700  4300
+U 5D59EC5C
 F0 "IO1" 50
 F1 "IO1.sch" 50
-F2 "A0" I R 5750 1250 50
-F3 "A1" I R 5750 1350 50
-F4 "A2" I R 5750 1450 50
-F5 "A3" I R 5750 1550 50
-F6 "A4" I R 5750 1650 50
-F7 "A5" I R 5750 1750 50
-F8 "A6" I R 5750 1850 50
-F9 "A7" I R 5750 1950 50
-F10 "A8" I R 5750 2050 50
-F11 "A9" I R 5750 2150 50
-F12 "A10" I R 5750 2250 50
-F13 "A11" I R 5750 2350 50
-F14 "A12" I R 5750 2450 50
-F15 "A13" I R 5750 2550 50
-F16 "A14" I R 5750 2650 50
-F17 "A15" I R 5750 2750 50
-F18 "~WR" I R 5750 3800 50
-F19 "~RD" I R 5750 3700 50
-F20 "+5V" I R 5750 1150 50
-F21 "GND" I R 5750 5250 50
-F22 "D0" I R 5750 2850 50
-F23 "D1" I R 5750 2950 50
-F24 "D2" I R 5750 3050 50
-F25 "D3" I R 5750 3150 50
-F26 "D4" I R 5750 3250 50
-F27 "D5" I R 5750 3350 50
-F28 "D6" I R 5750 3450 50
-F29 "D7" I R 5750 3550 50
-F30 "~IO0_CS" I R 5750 4000 50
-F31 "~IO1_CS" I R 5750 4100 50
-F32 "~IO2_CS" I R 5750 4200 50
-F33 "~IO3_CS" I R 5750 4300 50
-F34 "~IO4_CS" I R 5750 4400 50
-F35 "~IO5_CS" I R 5750 4500 50
-F36 "~IO6_CS" I R 5750 4600 50
-F37 "~IO7_CS" I R 5750 4700 50
-F38 "RESET" I R 5750 5150 50
+F2 "A0" I R 5650 1250 50
+F3 "A1" I R 5650 1350 50
+F6 "A4" I R 5650 1650 50
+F7 "A5" I R 5650 1750 50
+F8 "A6" I R 5650 1850 50
+F18 "~WR" I R 5650 3800 50
+F19 "~RD" I R 5650 3700 50
+F20 "+5V" I R 5650 1150 50
+F21 "GND" I R 5650 5250 50
+F22 "D0" I R 5650 2850 50
+F23 "D1" I R 5650 2950 50
+F24 "D2" I R 5650 3050 50
+F25 "D3" I R 5650 3150 50
+F26 "D4" I R 5650 3250 50
+F27 "D5" I R 5650 3350 50
+F28 "D6" I R 5650 3450 50
+F29 "D7" I R 5650 3550 50
+F30 "RESET" I R 5650 5150 50
+F31 "~IOREQ" I R 5650 3900 50
 $EndSheet
 $Sheet
@@
 F28 "D6" I R 6600 3450 50
 F29 "D7" I R 6600 3550 50
-F30 "~IO0_CS" I R 6600 4000 50
-F31 "~IO1_CS" I R 6600 4100 50
-F32 "~IO2_CS" I R 6600 4200 50
-F33 "~IO3_CS" I R 6600 4300 50
-F34 "~IO4_CS" I R 6600 4400 50
-F35 "~IO5_CS" I R 6600 4500 50
-F36 "~IO6_CS" I R 6600 4600 50
-F37 "~IO7_CS" I R 6600 4700 50
-F38 "RESET" I R 6600 5150 50
+F30 "~MEMRQ" I R 6600 4000 50
+$EndSheet
+$Sheet
+S 6750 1050 700  4300
+U 5D62F4AC
+F0 "ATA.sch" 50
+F1 "ATA.sch" 50
+F2 "A0" I R 7450 1250 50
+F3 "A1" I R 7450 1350 50
+F4 "A2" I R 7450 1450 50
+F6 "A4" I R 7450 1650 50
+F7 "A5" I R 7450 1750 50
+F8 "A6" I R 7450 1850 50
+F18 "~WR" I R 7450 3800 50
+F19 "~RD" I R 7450 3700 50
+F20 "+5V" I R 7450 1150 50
+F21 "GND" I R 7450 5250 50
+F22 "D0" I R 7450 2850 50
+F23 "D1" I R 7450 2950 50
+F24 "D2" I R 7450 3050 50
+F25 "D3" I R 7450 3150 50
+F26 "D4" I R 7450 3250 50
+F27 "D5" I R 7450 3350 50
+F28 "D6" I R 7450 3450 50
+F29 "D7" I R 7450 3550 50
+F30 "RESET" I R 7450 5150 50
+F31 "~IOREQ" I R 7450 3900 50
 $EndSheet
 $EndSCHEMATC

Commit message: 1
Changed lines of the file:
@@
 $EndDescr
-$Sheet
-S 3100 1050 700  4300
-U 5C68B4BB
-F0 "CPU" 50
-F1 "CPU.sch" 50
-F2 "A0" I R 3800 1250 50
-F3 "A1" I R 3800 1350 50
-F4 "A2" I R 3800 1450 50
-F5 "A3" I R 3800 1550 50
-F6 "A4" I R 3800 1650 50
-F7 "A5" I R 3800 1750 50
-F8 "A6" I R 3800 1850 50
-F9 "A7" I R 3800 1950 50
-F10 "A8" I R 3800 2050 50
-F11 "A9" I R 3800 2150 50
-F12 "A10" I R 3800 2250 50
-F13 "A11" I R 3800 2350 50
-F14 "A12" I R 3800 2450 50
-F15 "A13" I R 3800 2550 50
-F16 "A14" I R 3800 2650 50
-F17 "A15" I R 3800 2750 50
-F18 "~WR" I R 3800 3800 50
-F19 "~RD" I R 3800 3700 50
-F20 "+5V" I R 3800 1150 50
-F21 "GND" I R 3800 5250 50
-F22 "D0" I R 3800 2850 50
-F23 "D1" I R 3800 2950 50
-F24 "D2" I R 3800 3050 50
-F25 "D3" I R 3800 3150 50
-F26 "D4" I R 3800 3250 50
-F27 "D5" I R 3800 3350 50
-F28 "D6" I R 3800 3450 50
-F29 "D7" I R 3800 3550 50
-F30 "RESET" I R 3800 5150 50
-F31 "~IORQ" I R 3800 3900 50
-F32 "~MEMRQ" I R 3800 4000 50
-$EndSheet
 $Sheet
 S 4050 1050 700  4300
@@
 F17 "D6" I R 4750 3450 50
 F18 "D7" I R 4750 3550 50
-F19 "RESET" I R 4750 5150 50
-F20 "~IOREQ" I R 4750 3900 50
+F19 "~IORQ" I R 4750 3900 50
+F20 "RESET" I R 4750 5150 50
 $EndSheet
 $Sheet
@@
 F17 "D6" I R 5650 3450 50
 F18 "D7" I R 5650 3550 50
-F19 "RESET" I R 5650 5150 50
-F20 "~IOREQ" I R 5650 3900 50
+F19 "~IORQ" I R 5650 3900 50
+F20 "RESET" I R 5650 5150 50
 $EndSheet
 $Sheet
@@
 F0 "ATA.sch" 50
 F1 "ATA.sch" 50
-F2 "A0" I R 7450 1250 50
-F3 "A1" I R 7450 1350 50
-F4 "A2" I R 7450 1450 50
-F5 "A4" I R 7450 1650 50
-F6 "A5" I R 7450 1750 50
-F7 "A6" I R 7450 1850 50
-F8 "~WR" I R 7450 3800 50
-F9 "~RD" I R 7450 3700 50
-F10 "+5V" I R 7450 1150 50
-F11 "GND" I R 7450 5250 50
-F12 "D0" I R 7450 2850 50
-F13 "D1" I R 7450 2950 50
-F14 "D2" I R 7450 3050 50
-F15 "D3" I R 7450 3150 50
-F16 "D4" I R 7450 3250 50
-F17 "D5" I R 7450 3350 50
-F18 "D6" I R 7450 3450 50
-F19 "D7" I R 7450 3550 50
-F20 "RESET" I R 7450 5150 50
-F21 "~IOREQ" I R 7450 3900 50
+$EndSheet
+$Sheet
+S 3100 1050 700  4300
+U 5C68B4BB
+F0 "CPU" 50
+F1 "CPU.sch" 50
+F2 "A0" I R 3800 1250 50
+F3 "A1" I R 3800 1350 50
+F4 "A2" I R 3800 1450 50
+F5 "A3" I R 3800 1550 50
+F6 "A4" I R 3800 1650 50
+F7 "A5" I R 3800 1750 50
+F8 "A6" I R 3800 1850 50
+F9 "A7" I R 3800 1950 50
+F10 "A8" I R 3800 2050 50
+F11 "A9" I R 3800 2150 50
+F12 "A10" I R 3800 2250 50
+F13 "A11" I R 3800 2350 50
+F14 "A12" I R 3800 2450 50
+F15 "A13" I R 3800 2550 50
+F16 "A14" I R 3800 2650 50
+F17 "A15" I R 3800 2750 50
+F18 "~WR" I R 3800 3800 50
+F19 "~RD" I R 3800 3700 50
+F20 "+5V" I R 3800 1150 50
+F21 "GND" I R 3800 5250 50
+F22 "D0" I R 3800 2850 50
+F23 "D1" I R 3800 2950 50
+F24 "D2" I R 3800 3050 50
+F25 "D3" I R 3800 3150 50
+F26 "D4" I R 3800 3250 50
+F27 "D5" I R 3800 3350 50
+F28 "D6" I R 3800 3450 50
+F29 "D7" I R 3800 3550 50
+F30 "~IORQ" I R 3800 3900 50
+F31 "~MEMRQ" I R 3800 4000 50
+F33 "RESET" I R 3800 5150 50
 $EndSheet
 $EndSCHEMATC

Commit message: 123
Changed lines of the file:
@@
 F0 "ATA.sch" 50
 F1 "ATA.sch" 50
+F2 "GND" I R 7450 5250 50
+F3 "+5V" I R 7450 1150 50
+F4 "A6" I R 7450 1850 50
+F5 "A5" I R 7450 1750 50
+F6 "A4" I R 7450 1650 50
+F7 "~IOREQ" I R 7450 3900 50
+F8 "A1" I R 7450 1350 50
+F9 "A0" I R 7450 1250 50
+F10 "A2" I R 7450 1450 50
+F11 "~WR" I R 7450 3800 50
+F12 "~RD" I R 7450 3700 50
+F13 "~RESET" I R 7450 5000 50
+F14 "D1" I R 7450 2950 50
+F15 "D0" I R 7450 2850 50
+F16 "D2" I R 7450 3050 50
+F17 "D4" I R 7450 3250 50
+F18 "D3" I R 7450 3150 50
+F19 "D5" I R 7450 3350 50
+F20 "D6" I R 7450 3450 50
+F21 "D7" I R 7450 3550 50
 $EndSheet
 $Sheet
@@
 F30 "~IORQ" I R 3800 3900 50
 F31 "~MEMRQ" I R 3800 4000 50
-F33 "RESET" I R 3800 5150 50
+F32 "RESET" I R 3800 5150 50
 $EndSheet
 $EndSCHEMATC

Commit message: 1
Connections:
- net labels added: +5V, GND, RESET, ~A0, ~A1, ~A10, ~A11, ~A12, ~A13, ~A14, ~A15, ~A2, ~A3, ~A4, ~A5, ~A6, ~A7, ~A8, ~A9, ~D0, ~D1, ~D2, ~D3, ~D4, ~D5, ~D6, ~D7, ~IORQ, ~MEMRQ, ~RD, ~WR
- wire segments 0 -> 124
