File: Hardware/Project/ATA.sch (KiCad schematic (older format))
At the start: 9 parts, among them U10 ATA, U8 74LS138, U9 74LS14

Commit message: 1
Parts:
- removed U8: 74LS138, Package_DIP:DIP-16_W7.62mm_Socket, symbol 74xx:74LS138
- removed U9: 74LS14, Package_DIP:DIP-14_W7.62mm_Socket, symbol 74xx:74LS14
- added Q2: 9013, Package_TO_SOT_THT:TO-92, symbol Device:Q_NPN_CBE
- added R25: 47k, Resistor_SMD:R_0805_2012Metric, symbol Device:R
- R20: renamed from R1; value 1k -> 10k
- R21: renamed from R2; value 1k -> 10k
- R22: renamed from R3; value 1k -> 10k
- R23: renamed from R4; value 1k -> 10k
- R24: renamed from R5; value 1k -> 330
- U9: renamed from U10; footprint Package_DIP:DIP-40_W25.4mm_Socket -> Connector_PinHeader_2.54mm:PinHeader_2x20_P2.54mm_Vertical; symbol Vintage:ATA -> 8051-rescue:ATA-Vintage
- renumbered D1 to D10
Connections:
- net labels removed: A4, A5, A6, ~IO0_CS, ~IO1_CS, ~IO4_CS, ~IO5_CS, ~IO6_CS, ~IO7_CS, ~IOREQ
- wire segments 78 -> 60

Commit message: 1
Parts:
- added C9: 1uf, Capacitor_SMD:C_0805_2012Metric, symbol Device:C
Connections:
- wire segments 60 -> 65
Other:
- note added: "https://z80project.wordpress.com/2015/07/06/z80-8-bit-compact-flash-card-interface-part-1/"
- moved on the sheet: D10, Q2, R20, R21, R22, R23, R24, R25, U9
