File: Hardware/Project/Memory.sch (KiCad schematic (older format))
At the start: 3 parts, among them U10 28C256, U12 28C256, U9 7400

Commit message: 1
Parts:
- removed U9: 7400, symbol 74xx:7400
- added U?: 74LS138, symbol 74xx:74LS138
Connections:
- net +5V: now also U?.16 (VCC), U?.6 (E3)
- net A15: now also U?.1 (A0)
- net GND: now also U?.2 (A1), U?.3 (A2), U?.8 (GND)
- net ~MEM0_CS: now reaches U10.20 (~CS)
- net ~MEM0_CS: now also U?.15 (O0)
- net ~MEM1_CS: now reaches U12.20 (~CS)
- net ~MEM1_CS: now also U?.14 (O1)
- new net ~MEM2_CS: U?.13 (O2)
- new net ~MEM3_CS: U?.12 (O3)
- new net ~MEM4_CS: U?.11 (O4)
- new net ~MEM5_CS: U?.10 (O5)
- new net ~MEM6_CS: U?.9 (O6)
- new net ~MEM7_CS: U?.7 (O7)
- new net ~MEMRQ: U?.4 (E1), U?.5 (E2)
Other:
- moved on the sheet: U10, U12

Commit message: 1
Parts:
- gave numbers to parts that had none: 1
Changed lines of the file:
@@
 AR Path="/5DED3C2A/5D5D1AF9" Ref="U?"  Part="1"
 AR Path="/5D59EC5C/5D5D1AF9" Ref="U?"  Part="1"
-AR Path="/5E17A1DA/5D5D1AF9" Ref="U?"  Part="1"
-F 0 "U?" H 2500 3300 50  0000 C CNN
+AR Path="/5E17A1DA/5D5D1AF9" Ref="U18"  Part="1"
+F 0 "U18" H 2500 3300 50  0000 C CNN
 F 1 "74LS138" H 3000 3300 50  0000 C CNN
 F 2 "" H 2750 2850 50  0001 C CNN

Commit message: 1
Connections:
- net labels removed: ~MEM2_CS, ~MEM3_CS, ~MEM4_CS, ~MEM5_CS, ~MEM6_CS, ~MEM7_CS
Changed lines of the file:
@@
 $Descr A4 11693 8268
 encoding utf-8
-Sheet 5 6
+Sheet 4 6
 Title ""
 Date ""
@@
 Wire Wire Line
 	3350 2650 3250 2650
-Text GLabel 3350 2750 2    50   Input ~ 0
-~MEM2_CS
 Wire Wire Line
 	3350 2750 3250 2750
-Text GLabel 3350 2850 2    50   Input ~ 0
-~MEM3_CS
 Wire Wire Line
 	3350 2850 3250 2850
-Text GLabel 3350 2950 2    50   Input ~ 0
-~MEM4_CS
 Wire Wire Line
 	3350 2950 3250 2950
-Text GLabel 3350 3050 2    50   Input ~ 0
-~MEM5_CS
 Wire Wire Line
 	3350 3050 3250 3050
-Text GLabel 3350 3150 2    50   Input ~ 0
-~MEM6_CS
 Wire Wire Line
 	3350 3150 3250 3150
-Text GLabel 3350 3250 2    50   Input ~ 0
-~MEM7_CS
 Wire Wire Line
 	3350 3250 3250 3250

Commit message: 123
Parts:
- added U17: 28C256, Package_DIP:DIP-28_W15.24mm_Socket, symbol Memory_EEPROM:28C256
- U5: renamed from U18; footprint (none) -> Package_DIP:DIP-18_W7.62mm_Socket
- U6: renamed from U10; footprint (none) -> Package_DIP:DIP-32_W15.24mm_Socket
- U7: renamed from U12; footprint (none) -> Package_DIP:DIP-32_W15.24mm_Socket
Connections:
- net labels added: ~RD_BIOS, ~WR_BIOS
- wire segments 87 -> 117
Changed lines of the file:
@@
 Text HLabel 5500 1950 2    50   Input ~ 0
 D0
-Text HLabel 8850 4950 2    50   Input ~ 0
+Text HLabel 9300 4950 2    50   Input ~ 0
 GND
-Text HLabel 9050 950  2    50   Input ~ 0
+Text HLabel 9350 950  2    50   Input ~ 0
 +5V
 $Comp
-L Memory_EEPROM:28C256 U10
+L Memory_EEPROM:28C256 U6
 U 1 1 5E1802DB
 P 4850 2850
-F 0 "U10" H 4600 3900 50  0000 C CNN
+F 0 "U6" H 4600 3900 50  0000 C CNN
 F 1 "28C256" H 5100 3900 50  0000 C CNN
-F 2 "" H 4850 2850 50  0001 C CNN
+F 2 "Package_DIP:DIP-32_W15.24mm_Socket" H 4850 2850 50  0001 C CNN
 F 3 "http://ww1.microchip.com/downloads/en/DeviceDoc/doc0006.pdf" H 4850 2850 50  0001 C CNN
 	1    4850 2850
@@
 $EndComp
 $Comp
-L Memory_EEPROM:28C256 U12
+L Memory_EEPROM:28C256 U7
 U 1 1 5E180348
 P 6650 2850
-F 0 "U12" H 6400 3900 50  0000 C CNN
+F 0 "U7" H 6400 3900 50  0000 C CNN
 F 1 "28C256" H 6900 3900 50  0000 C CNN
-F 2 "" H 6650 2850 50  0001 C CNN
+F 2 "Package_DIP:DIP-32_W15.24mm_Socket" H 6650 2850 50  0001 C CNN
 F 3 "http://ww1.microchip.com/downloads/en/DeviceDoc/doc0006.pdf" H 6650 2850 50  0001 C CNN
 	1    6650 2850
@@
 AR Path="/5DED3C2A/5D5D1AF9" Ref="U?"  Part="1"
 AR Path="/5D59EC5C/5D5D1AF9" Ref="U?"  Part="1"
-AR Path="/5E17A1DA/5D5D1AF9" Ref="U18"  Part="1"
-F 0 "U18" H 2500 3300 50  0000 C CNN
+AR Path="/5E17A1DA/5D5D1AF9" Ref="U5"  Part="1"
+F 0 "U5" H 2500 3300 50  0000 C CNN
 F 1 "74LS138" H 3000 3300 50  0000 C CNN
-F 2 "" H 2750 2850 50  0001 C CNN
+F 2 "Package_DIP:DIP-18_W7.62mm_Socket" H 2750 2850 50  0001 C CNN
 F 3 "http://www.ti.com/lit/gpn/sn74LS138" H 2750 2850 50  0001 C CNN
 	1    2750 2850
@@
 Connection ~ 6650 4950
 Wire Wire Line
-	6650 4950 8850 4950
-Wire Wire Line
-	6650 950  9050 950
+	6650 4950 8800 4950
+Wire Wire Line
+	6650 950  8800 950
 Text GLabel 4200 3750 0    50   Input ~ 0
 ~MEM0_CS
@@
 Wire Wire Line
 	2750 3600 2750 4950
+$Comp
+L Memory_EEPROM:28C256 U?
+U 1 1 5DBEF611
+P 8800 2850
+AR Path="/5C68B4BB/5DBEF611" Ref="U?"  Part="1"
+AR Path="/5DED3C2A/5DBEF611" Ref="U?"  Part="1"
+AR Path="/5E17A1DA/5DBEF611" Ref="U17"  Part="1"
+F 0 "U17" H 8550 3900 50  0000 C CNN
+F 1 "28C256" H 9050 3900 50  0000 C CNN
+F 2 "Package_DIP:DIP-28_W15.24mm_Socket" H 8800 2850 50  0001 C CNN
+F 3 "http://ww1.microchip.com/downloads/en/DeviceDoc/doc0006.pdf" H 8800 2850 50  0001 C CNN
+	1    8800 2850
+	1    0    0    -1
+$EndComp
+Wire Wire Line
+	8400 3350 7750 3350
+Wire Wire Line
+	8400 3250 7750 3250
+Wire Wire Line
+	8400 3150 7750 3150
+Wire Wire Line
+	8400 3050 7750 3050
+Wire Wire Line
+	8400 2950 7750 2950
+Wire Wire Line
+	8400 2850 7750 2850
+Wire Wire Line
+	8400 2750 7750 2750
+Text HLabel 7750 3350 0    50   Input ~ 0
+A14
+Text HLabel 7750 3250 0    50   Input ~ 0
+A13
+Text HLabel 7750 3150 0    50   Input ~ 0
+A12
+Text HLabel 7750 3050 0    50   Input ~ 0
+A11
+Text HLabel 7750 2950 0    50   Input ~ 0
+A10
+Text HLabel 7750 2850 0    50   Input ~ 0
+A9
+Text HLabel 7750 2750 0    50   Input ~ 0
+A8
+Wire Wire Line
+	8400 2650 7750 2650
+Wire Wire Line
+	7750 2550 8400 2550
+Wire Wire Line
+	8400 2450 7750 2450
+Wire Wire Line
+	7750 2350 8400 2350
+Wire Wire Line
+	8400 2250 7750 2250
+Wire Wire Line
+	7750 2150 8400 2150
+Wire Wire Line
+	8400 2050 7750 2050
+Text HLabel 7750 2650 0    50   Input ~ 0
+A7
+Text HLabel 7750 2550 0    50   Input ~ 0
+A6
+Text HLabel 7750 2450 0    50   Input ~ 0
+A5
+Text HLabel 7750 2350 0    50   Input ~ 0
+A4
+Text HLabel 7750 2250 0    50   Input ~ 0
+A3
+Text HLabel 7750 2150 0    50   Input ~ 0
+A2
+Text HLabel 7750 2050 0    50   Input ~ 0
+A1
+Text HLabel 7750 1950 0    50   Input ~ 0
+A0
+Wire Wire Line
+	8400 1950 7750 1950
+Text HLabel 9350 2650 2    50   Input ~ 0
+D7
+Text HLabel 9350 2550 2    50   Input ~ 0
+D6
+Text HLabel 9350 2450 2    50   Input ~ 0
+D5
+Text HLabel 9350 2350 2    50   Input ~ 0
+D4
+Text HLabel 9350 2250 2    50   Input ~ 0
+D3
+Text HLabel 9350 2150 2    50   Input ~ 0
+D2
+Text HLabel 9350 2050 2    50   Input ~ 0
+D1
+Text HLabel 9350 1950 2    50   Input ~ 0
+D0
+Wire Wire Line
+	9350 1950 9200 1950
+Wire Wire Line
+	9350 2050 9200 2050
+Wire Wire Line
+	9350 2150 9200 2150
+Wire Wire Line
+	9350 2250 9200 2250
+Wire Wire Line
+	9350 2350 9200 2350
+Wire Wire Line
+	9350 2450 9200 2450
+Wire Wire Line
+	9350 2550 9200 2550
+Wire Wire Line
+	9350 2650 9200 2650
+Wire Wire Line
+	7750 3550 8400 3550
+Wire Wire Line
+	8400 3650 7750 3650
+Wire Wire Line
+	8800 950  8800 1750
+Text HLabel 7750 3750 0    50   Input ~ 0
+~MEMRQ
+Wire Wire Line
+	8800 3950 8800 4950
+Wire Wire Line
+	7750 3750 8400 3750
+Text HLabel 7750 3650 0    50   Input ~ 0
+~RD_BIOS
+Text HLabel 7750 3550 0    50   Input ~ 0
+~WR_BIOS
+Connection ~ 8800 950
+Connection ~ 8800 4950
+Wire Wire Line
+	8800 4950 9300 4950
+Wire Wire Line
+	8800 950  9350 950
 $EndSCHEMATC

Commit message: 1
Parts:
- removed U17: 28C256, Package_DIP:DIP-28_W15.24mm_Socket, symbol Memory_EEPROM:28C256
- U5: footprint Package_DIP:DIP-18_W7.62mm_Socket -> Package_DIP:DIP-16_W7.62mm_Socket
Connections:
- net labels removed: ~RD_BIOS, ~WR_BIOS
- wire segments 117 -> 87
Changed lines of the file:
@@
 $Descr A4 11693 8268
 encoding utf-8
-Sheet 4 6
+Sheet 3 5
 Title ""
 Date ""
@@
 F 0 "U5" H 2500 3300 50  0000 C CNN
 F 1 "74LS138" H 3000 3300 50  0000 C CNN
-F 2 "Package_DIP:DIP-18_W7.62mm_Socket" H 2750 2850 50  0001 C CNN
+F 2 "Package_DIP:DIP-16_W7.62mm_Socket" H 2750 2850 50  0001 C CNN
 F 3 "http://www.ti.com/lit/gpn/sn74LS138" H 2750 2850 50  0001 C CNN
 	1    2750 2850
@@
 Connection ~ 6650 950
 Connection ~ 6650 4950
-Wire Wire Line
-	6650 4950 8800 4950
-Wire Wire Line
-	6650 950  8800 950
 Text GLabel 4200 3750 0    50   Input ~ 0
 ~MEM0_CS
@@
 Wire Wire Line
 	2750 3600 2750 4950
-$Comp
-L Memory_EEPROM:28C256 U?
-U 1 1 5DBEF611
-P 8800 2850
-AR Path="/5C68B4BB/5DBEF611" Ref="U?"  Part="1"
-AR Path="/5DED3C2A/5DBEF611" Ref="U?"  Part="1"
-AR Path="/5E17A1DA/5DBEF611" Ref="U17"  Part="1"
-F 0 "U17" H 8550 3900 50  0000 C CNN
-F 1 "28C256" H 9050 3900 50  0000 C CNN
-F 2 "Package_DIP:DIP-28_W15.24mm_Socket" H 8800 2850 50  0001 C CNN
-F 3 "http://ww1.microchip.com/downloads/en/DeviceDoc/doc0006.pdf" H 8800 2850 50  0001 C CNN
-	1    8800 2850
-	1    0    0    -1
-$EndComp
-Wire Wire Line
-	8400 3350 7750 3350
-Wire Wire Line
-	8400 3250 7750 3250
-Wire Wire Line
-	8400 3150 7750 3150
-Wire Wire Line
-	8400 3050 7750 3050
-Wire Wire Line
-	8400 2950 7750 2950
-Wire Wire Line
-	8400 2850 7750 2850
-Wire Wire Line
-	8400 2750 7750 2750
-Text HLabel 7750 3350 0    50   Input ~ 0
-A14
-Text HLabel 7750 3250 0    50   Input ~ 0
-A13
-Text HLabel 7750 3150 0    50   Input ~ 0
-A12
-Text HLabel 7750 3050 0    50   Input ~ 0
-A11
-Text HLabel 7750 2950 0    50   Input ~ 0
-A10
-Text HLabel 7750 2850 0    50   Input ~ 0
-A9
-Text HLabel 7750 2750 0    50   Input ~ 0
-A8
-Wire Wire Line
-	8400 2650 7750 2650
-Wire Wire Line
-	7750 2550 8400 2550
-Wire Wire Line
-	8400 2450 7750 2450
-Wire Wire Line
-	7750 2350 8400 2350
-Wire Wire Line
-	8400 2250 7750 2250
-Wire Wire Line
-	7750 2150 8400 2150
-Wire Wire Line
-	8400 2050 7750 2050
-Text HLabel 7750 2650 0    50   Input ~ 0
-A7
-Text HLabel 7750 2550 0    50   Input ~ 0
-A6
-Text HLabel 7750 2450 0    50   Input ~ 0
-A5
-Text HLabel 7750 2350 0    50   Input ~ 0
-A4
-Text HLabel 7750 2250 0    50   Input ~ 0
-A3
-Text HLabel 7750 2150 0    50   Input ~ 0
-A2
-Text HLabel 7750 2050 0    50   Input ~ 0
-A1
-Text HLabel 7750 1950 0    50   Input ~ 0
-A0
-Wire Wire Line
-	8400 1950 7750 1950
-Text HLabel 9350 2650 2    50   Input ~ 0
-D7
-Text HLabel 9350 2550 2    50   Input ~ 0
-D6
-Text HLabel 9350 2450 2    50   Input ~ 0
-D5
-Text HLabel 9350 2350 2    50   Input ~ 0
-D4
-Text HLabel 9350 2250 2    50   Input ~ 0
-D3
-Text HLabel 9350 2150 2    50   Input ~ 0
-D2
-Text HLabel 9350 2050 2    50   Input ~ 0
-D1
-Text HLabel 9350 1950 2    50   Input ~ 0
-D0
-Wire Wire Line
-	9350 1950 9200 1950
-Wire Wire Line
-	9350 2050 9200 2050
-Wire Wire Line
-	9350 2150 9200 2150
-Wire Wire Line
-	9350 2250 9200 2250
-Wire Wire Line
-	9350 2350 9200 2350
-Wire Wire Line
-	9350 2450 9200 2450
-Wire Wire Line
-	9350 2550 9200 2550
-Wire Wire Line
-	9350 2650 9200 2650
-Wire Wire Line
-	7750 3550 8400 3550
-Wire Wire Line
-	8400 3650 7750 3650
-Wire Wire Line
-	8800 950  8800 1750
-Text HLabel 7750 3750 0    50   Input ~ 0
-~MEMRQ
-Wire Wire Line
-	8800 3950 8800 4950
-Wire Wire Line
-	7750 3750 8400 3750
-Text HLabel 7750 3650 0    50   Input ~ 0
-~RD_BIOS
-Text HLabel 7750 3550 0    50   Input ~ 0
-~WR_BIOS
-Connection ~ 8800 950
-Connection ~ 8800 4950
-Wire Wire Line
-	8800 4950 9300 4950
-Wire Wire Line
-	8800 950  9350 950
+Wire Wire Line
+	6650 950  9350 950
+Wire Wire Line
+	6650 4950 9300 4950
 $EndSCHEMATC

Commit message: 1
Parts:
- added C6, C7, C8: 1uf, Capacitor_SMD:C_0805_2012Metric, symbol Device:C
- U6, U7: footprint Package_DIP:DIP-32_W15.24mm_Socket -> Package_DIP:DIP-28_W15.24mm_Socket
Connections:
- wire segments 87 -> 102
Changed lines of the file:
@@
 F 0 "U6" H 4600 3900 50  0000 C CNN
 F 1 "28C256" H 5100 3900 50  0000 C CNN
-F 2 "Package_DIP:DIP-32_W15.24mm_Socket" H 4850 2850 50  0001 C CNN
+F 2 "Package_DIP:DIP-28_W15.24mm_Socket" H 4850 2850 50  0001 C CNN
 F 3 "http://ww1.microchip.com/downloads/en/DeviceDoc/doc0006.pdf" H 4850 2850 50  0001 C CNN
 	1    4850 2850
@@
 F 0 "U7" H 6400 3900 50  0000 C CNN
 F 1 "28C256" H 6900 3900 50  0000 C CNN
-F 2 "Package_DIP:DIP-32_W15.24mm_Socket" H 6650 2850 50  0001 C CNN
+F 2 "Package_DIP:DIP-28_W15.24mm_Socket" H 6650 2850 50  0001 C CNN
 F 3 "http://ww1.microchip.com/downloads/en/DeviceDoc/doc0006.pdf" H 6650 2850 50  0001 C CNN
 	1    6650 2850
@@
 	4850 950  2750 950
 Wire Wire Line
-	2750 950  2750 2200
+	2750 950  2750 1150
 Connection ~ 4850 950
 Wire Wire Line
-	4850 950  4850 1750
-Wire Wire Line
-	6650 950  6650 1750
+	4850 950  4850 1150
+Wire Wire Line
+	6650 950  6650 1150
 Connection ~ 6650 950
 Connection ~ 6650 4950
@@
 Wire Wire Line
 	6650 4950 9300 4950
+$Comp
+L Device:C C?
+U 1 1 5D172A2A
+P 6900 1350
+AR Path="/5D172A2A" Ref="C?"  Part="1"
+AR Path="/5C68B4BB/5D172A2A" Ref="C?"  Part="1"
+AR Path="/5C8BEFCF/5D172A2A" Ref="C?"  Part="1"
+AR Path="/5DED3C2A/5D172A2A" Ref="C?"  Part="1"
+AR Path="/5E17A1DA/5D172A2A" Ref="C8"  Part="1"
+F 0 "C8" V 6950 1450 50  0000 L CNN
+F 1 "1uf" V 6950 1200 50  0000 L CNN
+F 2 "Capacitor_SMD:C_0805_2012Metric" H 6938 1200 50  0001 C CNN
+F 3 "~" H 6900 1350 50  0001 C CNN
+	1    6900 1350
+	-1   0    0    -1
+$EndComp
+Text HLabel 6950 1550 2    50   Input ~ 0
+GND
+Wire Wire Line
+	6900 1500 6900 1550
+Wire Wire Line
+	6900 1550 6950 1550
+Wire Wire Line
+	6900 1200 6900 1150
+Wire Wire Line
+	6900 1150 6650 1150
+Connection ~ 6650 1150
+Wire Wire Line
+	6650 1150 6650 1750
+$Comp
+L Device:C C?
+U 1 1 5D17D24F
+P 5100 1350
+AR Path="/5D17D24F" Ref="C?"  Part="1"
+AR Path="/5C68B4BB/5D17D24F" Ref="C?"  Part="1"
+AR Path="/5C8BEFCF/5D17D24F" Ref="C?"  Part="1"
+AR Path="/5DED3C2A/5D17D24F" Ref="C?"  Part="1"
+AR Path="/5E17A1DA/5D17D24F" Ref="C7"  Part="1"
+F 0 "C7" V 5150 1450 50  0000 L CNN
+F 1 "1uf" V 5150 1200 50  0000 L CNN
+F 2 "Capacitor_SMD:C_0805_2012Metric" H 5138 1200 50  0001 C CNN
+F 3 "~" H 5100 1350 50  0001 C CNN
+	1    5100 1350
+	-1   0    0    -1
+$EndComp
+Text HLabel 5150 1550 2    50   Input ~ 0
+GND
+Wire Wire Line
+	5100 1500 5100 1550
+Wire Wire Line
+	5100 1550 5150 1550
+Wire Wire Line
+	5100 1200 5100 1150
+Wire Wire Line
+	5100 1150 4850 1150
+Connection ~ 4850 1150
+Wire Wire Line
+	4850 1150 4850 1750
+$Comp
+L Device:C C?
+U 1 1 5D18843B
+P 3000 1350
+AR Path="/5D18843B" Ref="C?"  Part="1"
+AR Path="/5C68B4BB/5D18843B" Ref="C?"  Part="1"
+AR Path="/5C8BEFCF/5D18843B" Ref="C?"  Part="1"
+AR Path="/5DED3C2A/5D18843B" Ref="C?"  Part="1"
+AR Path="/5E17A1DA/5D18843B" Ref="C6"  Part="1"
+F 0 "C6" V 3050 1450 50  0000 L CNN
+F 1 "1uf" V 3050 1200 50  0000 L CNN
+F 2 "Capacitor_SMD:C_0805_2012Metric" H 3038 1200 50  0001 C CNN
+F 3 "~" H 3000 1350 50  0001 C CNN
+	1    3000 1350
+	-1   0    0    -1
+$EndComp
+Text HLabel 3050 1550 2    50   Input ~ 0
+GND
+Wire Wire Line
+	3000 1500 3000 1550
+Wire Wire Line
+	3000 1550 3050 1550
+Wire Wire Line
+	3000 1200 3000 1150
+Wire Wire Line
+	3000 1150 2750 1150
+Connection ~ 2750 1150
+Wire Wire Line
+	2750 1150 2750 2200
 $EndSCHEMATC
