File: Hardware/Project/8051.kicad_pcb (KiCad board)
At the start: 2 copper layers, 43 parts, among them Q1 Q_PNP_CBE, SW1 SW_Push, U1 8255, U10 ATA, U11 74LS138, U12 74LS08, U13 74LS00, U14 STC89C52, U15 74LS32, U16 74LS373, U17 28C256, U18 74LS30, U19 74LS32, U2 74LS138, U20 74LS138, U3 8255, U4 74LS138, U5 74LS138, U6 28C256, U7 28C256, U8 74LS138, U9 74LS14, Y1 Crystal, Y2 Crystal

Commit message: 1
Parts:
- removed C5, C6: C, Capacitor_SMD:C_0805_2012Metric
- removed R4, R5, R6, R8, R9: 1k, Resistor_SMD:R_0805_2012Metric
- removed R7: 1M, Resistor_SMD:R_0805_2012Metric
- removed U15: 74LS32, Package_DIP:DIP-14_W7.62mm_Socket
- removed U16: 74LS373, Package_DIP:DIP-20_W7.62mm_Socket
- removed U17: 28C256, Package_DIP:DIP-28_W15.24mm_Socket
- removed U3: 8255, Package_DIP:DIP-40_W15.24mm
- removed U4, U8: 74LS138, Package_DIP:DIP-18_W7.62mm_Socket
- removed Y1: Crystal, Connector_PinSocket_2.54mm:PinSocket_1x02_P2.54mm_Vertical
- added C1: CP1, Capacitor_THT:CP_Radial_D7.5mm_P2.50mm, F.Cu at (-321.6, -43.7)
- added D10: LED, LED_SMD:LED_0805_2012Metric, F.Cu at (-310.4, -13.2)
- added D3: ~ISP, LED_SMD:LED_0805_2012Metric, F.Cu at (-314.6, -39.5)
- added D4: POWER, LED_SMD:LED_0805_2012Metric, F.Cu at (-313.8, -34.8)
- added J1: USB_B_Mini, Connector_USB:USB_Micro-B_Wuerth_629105150521_CircularHoles, F.Cu at (-330.2, -46.2)
- added J2: Conn_02x20_Odd_Even, Connector_PinHeader_2.54mm:PinHeader_2x20_P2.54mm_Vertical, F.Cu at (-355.0, 46.2)
- added JP1: , Jumper:SolderJumper-2_P1.3mm_Open_RoundedPad1.0x1.5mm, F.Cu at (-391.9, 26.4)
- added JP2: , Jumper:SolderJumper-2_P1.3mm_Open_RoundedPad1.0x1.5mm, F.Cu at (-391.9, 29.0)
- added Q2: 9013, Package_TO_SOT_THT:TO-92, F.Cu at (-307.8, -9.65)
- added R13: 330, Resistor_SMD:R_0805_2012Metric, F.Cu at (-337.8, -37.6)
- added R14: 330, Resistor_SMD:R_0805_2012Metric, F.Cu at (-308.0, -39.6)
- added R15: 330, Resistor_SMD:R_0805_2012Metric, F.Cu at (-310.4, -34.9)
- added R20: 10k, Resistor_SMD:R_0805_2012Metric, F.Cu at (-310.4, -23.4)
- added R21: 10k, Resistor_SMD:R_0805_2012Metric, F.Cu at (-310.4, -21.3)
- added R22: 10k, Resistor_SMD:R_0805_2012Metric, F.Cu at (-310.4, -19.3)
- added R23: 10k, Resistor_SMD:R_0805_2012Metric, F.Cu at (-310.4, -17.3)
- added R24: 330, Resistor_SMD:R_0805_2012Metric, F.Cu at (-310.4, -15.2)
- added R25: 47k, Resistor_SMD:R_0805_2012Metric, F.Cu at (-374.8, -29.5)
- added U21: 74LS32, Package_DIP:DIP-14_W7.62mm_Socket, F.Cu at (-351.5, -10.2)
- added U22: 74LS138, Package_DIP:DIP-16_W7.62mm_Socket, F.Cu at (-354.1, 1.02)
- C2: value C -> CP1; footprint Capacitor_SMD:C_0805_2012Metric -> Capacitor_THT:CP_Radial_D7.5mm_P2.50mm
- C3: value CP1 -> C; footprint Capacitor_THT:CP_Radial_D4.0mm_P1.50mm -> Capacitor_SMD:C_0805_2012Metric
- D1: value LED -> DIODE
- D2: value DIODE -> ~BOOTING
- Q1: value Q_PNP_CBE -> 9015; footprint Button_Switch_Keyboard:SW_Cherry_MX1A_1.00u_PCB -> Package_TO_SOT_THT:TO-92
- SW1: value SW_Push -> reset; footprint Connector_PinSocket_2.54mm:PinSocket_1x02_P2.54mm_Vertical -> Button_Switch_THT:SW_PUSH_6mm
- U10: value ATA -> 74LS138; footprint Package_DIP:DIP-40_W25.4mm_Socket -> Package_DIP:DIP-16_W7.62mm_Socket
- U11: value 74LS138 -> 74LS14; footprint Package_DIP:DIP-18_W7.62mm_Socket -> Package_DIP:DIP-14_W7.62mm_Socket
- U12: value 74LS08 -> 74LS00
- U13: value 74LS00 -> STC89C52-Vintage; footprint Package_DIP:DIP-14_W7.62mm_Socket -> Package_DIP:DIP-40_W15.24mm_Socket
- U14: value STC89C52 -> 74LS08; footprint Package_DIP:DIP-40_W25.4mm_Socket -> Package_DIP:DIP-14_W7.62mm_Socket
- U18: value 74LS30 -> 74LS32
- U19: value 74LS32 -> 74LS30
- U2: value 74LS138 -> 74LS373_ARRANGED; footprint Package_DIP:DIP-18_W7.62mm_Socket -> Package_DIP:DIP-20_W7.62mm_Socket
- U20: value 74LS138 -> AT29C512; footprint Package_DIP:DIP-16_W7.62mm_Socket -> Package_DIP:DIP-32_W15.24mm_Socket
- U5: footprint Package_DIP:DIP-18_W7.62mm_Socket -> Package_DIP:DIP-16_W7.62mm_Socket
- U9: value 74LS14 -> ATA; footprint Package_DIP:DIP-14_W7.62mm_Socket -> Connector_PinHeader_2.54mm:PinHeader_2x20_P2.54mm_Vertical
- Y2: footprint Connector_PinSocket_2.54mm:PinSocket_1x02_P2.54mm_Vertical -> Crystal:Crystal_HC18-U_Vertical
- moved U5 654.2 mm to (-380.5, 24.9)
- moved U7 590.9 mm to (-354.1, 42.7), turned to 180 degrees
- moved U6 553.2 mm to (-334.8, 42.7), turned to 180 degrees
- moved R3 545.1 mm to (-361.6, -42.2)
- moved R1 543.8 mm to (-357.6, -41.7)
- moved R2 535.3 mm to (-356.0, -47.2)
- moved D1 513.8 mm to (-360.6, -47.2)
- moved U1 506.7 mm to (-388.6, 41.7), turned to 180 degrees
- moved U19 503.3 mm to (-403.5, -29.1), turned to 90 degrees
- moved U2 495.4 mm to (-357.6, -6.60), turned to 270 degrees
- moved C4 477.9 mm to (-395.9, -16.3), turned to 270 degrees
- moved U9 465.9 mm to (-308.4, 44.2), turned to 180 degrees
- moved U10 457.4 mm to (-332.2, 1.02), turned to 90 degrees
- moved Y2 455.9 mm to (-395.9, -21.1), turned to 180 degrees
- moved C3 452.5 mm to (-400.9, -16.3), turned to 270 degrees
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Connections:
- net /ATA.sch/D3 renamed Net-(U10-Pad11)
- net /ATA.sch/D4 renamed Net-(U10-Pad9)
- net /ATA.sch/D5 renamed Net-(U10-Pad7)
- net /CPU/~MEMRQ renamed Net-(U9-Pad4)
- C2 pad 1: Net-(C2-Pad1) -> ~RESET
- C2 pad 2: Net-(C2-Pad2) -> /GND
- C3 pad 1: ~RESET -> Net-(C3-Pad1)
- C3 pad 2: /CPU/GND -> /GND
- C4 pad 2: Net-(C2-Pad2) -> /GND
- D1 pad 1: Net-(D1-Pad1) -> ~RESET
- D1 pad 2: Net-(D1-Pad2) -> ~WARM_BOOT
- D2 pad 1: ~RESET -> ~BOOTING
- D2 pad 2: ~WARM_BOOT -> Net-(D2-Pad2)
- Q1 pad 1: /CPU/GND -> /GND
- R1 pad 1: /ATA.sch/+5V -> ~WARM_BOOT
- R1 pad 2: Net-(R1-Pad2) -> Net-(Q1-Pad2)
- R10 pad 1: /CPU/+5V -> /+5V
- R11 pad 1: Net-(C4-Pad1) -> /+5V
- R11 pad 2: Net-(R11-Pad2) -> ~ENTER_ISP
- R2 pad 1: /ATA.sch/+5V -> /+5V
- R2 pad 2: Net-(R2-Pad2) -> ~RESET
- R3 pad 1: /ATA.sch/+5V -> Net-(R3-Pad1)
- R3 pad 2: Net-(R3-Pad2) -> /GND
- RN1 pad 1: /CPU/+5V -> /+5V
- RN1 pad 2: /CPU/D0 -> /~D0
- RN1 pad 3: /CPU/D1 -> /~D1
- RN1 pad 4: /CPU/D2 -> /~D2
- RN1 pad 5: /CPU/D3 -> /~D3
- RN1 pad 6: /CPU/D4 -> /~D4
- RN1 pad 7: /CPU/D5 -> /~D5
- RN1 pad 8: /CPU/D6 -> /~D6
- RN1 pad 9: /CPU/D7 -> /~D7
- SW1 pad 1: /CPU/GND -> /GND
- U1 pad 26: /IO0/+5V -> /+5V
- U1 pad 27: /IO0/D7 -> /~D7
- U1 pad 28: /IO0/D6 -> /~D6
- U1 pad 29: /IO0/D5 -> /~D5
- U1 pad 30: /IO0/D4 -> /~D4
- U1 pad 31: /IO0/D3 -> /~D3
- U1 pad 32: /IO0/D2 -> /~D2
- U1 pad 33: /IO0/D1 -> /~D1
- U1 pad 34: /IO0/D0 -> /~D0
- U1 pad 35: /IO0/RESET -> /RESET
- U1 pad 36: /IO0/~WR -> /~WR
- U1 pad 5: /IO0/~RD -> /~RD
- U1 pad 6: ~IO0_CS -> Net-(JP1-Pad2)
- U1 pad 7: /IO0/GND -> /GND
- U1 pad 8: /IO0/A1 -> /~A1
- U1 pad 9: /IO0/A0 -> /~A0
- U10 pad 1: Net-(U10-Pad1) -> /~A0
- U10 pad 13: /ATA.sch/D2 -> ~WARM_BOOT
- U10 pad 14: Net-(U10-Pad14) -> ~ENTER_ISP
- U10 pad 15: /ATA.sch/D1 -> ~ENTER_ISP
- U10 pad 16: Net-(U10-Pad16) -> /+5V
- U10 pad 2: /ATA.sch/GND -> /~A1
- U10 pad 3: /ATA.sch/D7 -> /~A2
- U10 pad 4: Net-(U10-Pad4) -> ~IO7_CS
- U10 pad 5: /ATA.sch/D6 -> ~CPU_WR
- U10 pad 6: Net-(U10-Pad6) -> /+5V
- U10 pad 8: Net-(U10-Pad8) -> /GND
- U11 pad 1: /CPU/A0 -> ~RESET
- U11 pad 10: Net-(U11-Pad10) -> (no net)
- U11 pad 11: Net-(U11-Pad11) -> (no net)
- U11 pad 12: Net-(U11-Pad12) -> (no net)
- U11 pad 13: ~WARM_BOOT -> (no net)
- U11 pad 14: ~ENTER_ISP -> /+5V
- U11 pad 2: /CPU/A1 -> /RESET
- U11 pad 3: /CPU/A2 -> /~IORQ
- U11 pad 4: ~IO7_CS -> /~MEMRQ
- U11 pad 5: ~CPU_WR -> (no net)
- U11 pad 6: /CPU/+5V -> (no net)
- U11 pad 7: Net-(U11-Pad7) -> /GND
- U11 pad 8: Net-(C2-Pad2) -> (no net)
- U11 pad 9: Net-(U11-Pad9) -> (no net)
- U12 pad 1: ~CPU_RD -> ~ENTER_ISP
- U12 pad 10: (no net) -> ~ISP
- U12 pad 11: (no net) -> ~ISP
- U12 pad 12: (no net) -> ISP
- U12 pad 13: (no net) -> Net-(U12-Pad13)
- U12 pad 14: /CPU/+5V -> /+5V
- U12 pad 2: ~PSEN -> BOOTING
- U12 pad 3: Net-(U12-Pad3) -> ~BOOTING
- U12 pad 4: (no net) -> ~BOOTING
- U12 pad 5: (no net) -> ~RESET
- U12 pad 6: (no net) -> BOOTING
- U12 pad 7: Net-(C2-Pad2) -> /GND
- U12 pad 8: (no net) -> ISP
- U12 pad 9: (no net) -> ~ENTER_ISP
- U13 pad 1: ~ENTER_ISP -> Net-(U13-Pad1)
- U13 pad 10: ~ISP -> Net-(U13-Pad10)
- U13 pad 11: ~ISP -> Net-(U13-Pad11)
- U13 pad 12: ISP -> Net-(U13-Pad12)
- U13 pad 13: ~RESET -> Net-(U13-Pad13)
- U13 pad 14: /CPU/+5V -> Net-(U13-Pad14)
- U13 pad 2: BOOTING -> Net-(U13-Pad2)
- U13 pad 3: ~BOOTING -> Net-(U13-Pad3)
- U13 pad 4: ~BOOTING -> Net-(U13-Pad4)
- U13 pad 5: ~RESET -> Net-(U13-Pad5)
- U13 pad 6: BOOTING -> Net-(U13-Pad6)
- U13 pad 7: Net-(C2-Pad2) -> Net-(U13-Pad7)
- U13 pad 8: ISP -> Net-(U13-Pad8)
- U13 pad 9: ~ENTER_ISP -> /RESET
- U14 pad 1: Net-(U14-Pad1) -> Net-(U13-Pad29)
- U14 pad 10: Net-(U14-Pad10) -> (no net)
- U14 pad 11: Net-(U14-Pad11) -> (no net)
- U14 pad 12: Net-(U14-Pad12) -> (no net)
- U14 pad 13: Net-(U14-Pad13) -> (no net)
- U14 pad 14: Net-(U14-Pad14) -> /+5V
- U14 pad 2: Net-(U14-Pad2) -> Net-(U13-Pad17)
- U14 pad 3: Net-(U14-Pad3) -> ~CPU_RD
- U14 pad 4: Net-(U14-Pad4) -> (no net)
- U14 pad 5: Net-(U14-Pad5) -> (no net)
- U14 pad 6: Net-(U14-Pad6) -> (no net)
- U14 pad 7: Net-(U14-Pad7) -> /GND
- U14 pad 8: Net-(U14-Pad8) -> (no net)
- U14 pad 9: /CPU/RESET -> (no net)
- U18 pad 1: /CPU/A8 -> ~ISP
- U18 pad 10: (no net) -> ~CPU_WR
- U18 pad 11: /CPU/A14 -> /~RD
- U18 pad 12: /CPU/A15 -> BOOTING
- U18 pad 13: (no net) -> ~CPU_RD
- U18 pad 14: /CPU/+5V -> /+5V
- U18 pad 2: /CPU/A9 -> ~CPU_WR
- U18 pad 3: /CPU/A10 -> ~WR_BIOS
- U18 pad 4: /CPU/A11 -> ~BOOTING
- U18 pad 5: /CPU/A12 -> ~CPU_RD
- U18 pad 6: /CPU/A13 -> ~RD_BIOS
- U18 pad 7: Net-(U18-Pad7) -> /GND
- U18 pad 8: Net-(U18-Pad8) -> /~WR
- U18 pad 9: (no net) -> ISP
- U19 pad 1: /CPU/A7 -> /~A8
- U19 pad 11: (no net) -> /~A14
- U19 pad 12: (no net) -> /~A15
- U19 pad 14: /CPU/+5V -> /+5V
- U19 pad 2: Net-(U18-Pad8) -> /~A9
- U19 pad 3: /CPU/~IORQ -> /~A10
- U19 pad 4: (no net) -> /~A11
- U19 pad 5: (no net) -> /~A12
- U19 pad 6: (no net) -> /~A13
- U19 pad 7: Net-(C2-Pad2) -> /GND
- U19 pad 8: (no net) -> Net-(U19-Pad8)
- U2 pad 1: /IO0/A4 -> /GND
- U2 pad 10: Net-(U2-Pad10) -> /GND
- U2 pad 11: Net-(U2-Pad11) -> Net-(U13-Pad30)
- U2 pad 12: Net-(U2-Pad12) -> /~A7
- U2 pad 13: Net-(U2-Pad13) -> /~D7
- U2 pad 14: Net-(U2-Pad14) -> /~D5
- U2 pad 15: ~IO0_CS -> /~A5
- U2 pad 16: Net-(U2-Pad16) -> /~A3
- U2 pad 17: (no net) -> /~D3
- U2 pad 18: (no net) -> /~D1
- U2 pad 2: /IO0/A5 -> /~A0
- U2 pad 3: /IO0/A6 -> /~D0
- U2 pad 4: /IO0/~IORQ -> /~D2
- U2 pad 5: /IO0/~IORQ -> /~A2
- U2 pad 6: Net-(U2-Pad16) -> /~A4
- U2 pad 7: Net-(U2-Pad7) -> /~D4
- U2 pad 8: Net-(U2-Pad8) -> /~D6
- U2 pad 9: Net-(U2-Pad9) -> /~A6
- U20 pad 1: /CPU/A4 -> (no net)
- U20 pad 10: ~IO5_CS -> /~A2
- U20 pad 11: ~IO4_CS -> /~A1
- U20 pad 12: ~IO3_CS -> /~A0
- U20 pad 13: ~IO2_CS -> /~D0
- U20 pad 14: ~IO1_CS -> /~D1
- U20 pad 15: ~IO0_CS -> /~D2
- U20 pad 16: /CPU/+5V -> /GND
- U20 pad 2: /CPU/A5 -> (no net)
- U20 pad 3: /CPU/A6 -> /~A15
- U20 pad 4: /CPU/~IORQ -> /~A12
- U20 pad 5: /CPU/~IORQ -> /~A7
- U20 pad 6: /CPU/+5V -> /~A6
- U20 pad 7: ~IO7_CS -> /~A5
- U20 pad 8: /CPU/GND -> /~A4
- U20 pad 9: ~IO6_CS -> /~A3
- U5 pad 1: /Memory/A15 -> /~A15
- U5 pad 16: /Memory/+5V -> /+5V
- U5 pad 2: /Memory/GND -> /GND
- U5 pad 3: /Memory/GND -> /GND
- U5 pad 4: /Memory/~MEMRQ -> /~MEMRQ
- U5 pad 5: /Memory/~MEMRQ -> /~MEMRQ
- U5 pad 6: /Memory/+5V -> /+5V
- U5 pad 8: /Memory/GND -> /GND
- U6 pad 1: /Memory/A14 -> /~A14
- U6 pad 10: /Memory/A0 -> /~A0
- U6 pad 11: /Memory/D0 -> /~D0
- U6 pad 12: /Memory/D1 -> /~D1
- U6 pad 13: /Memory/D2 -> /~D2
- U6 pad 14: /Memory/GND -> /GND
- U6 pad 15: /Memory/D3 -> /~D3
- U6 pad 16: /Memory/D4 -> /~D4
- U6 pad 17: /Memory/D5 -> /~D5
- U6 pad 18: /Memory/D6 -> /~D6
- U6 pad 19: /Memory/D7 -> /~D7
- U6 pad 2: /Memory/A12 -> /~A12
- U6 pad 21: /Memory/A10 -> /~A10
- U6 pad 22: /Memory/~RD -> /~RD
- U6 pad 23: /Memory/A11 -> /~A11
- U6 pad 24: /Memory/A9 -> /~A9
- U6 pad 25: /Memory/A8 -> /~A8
- U6 pad 26: /Memory/A13 -> /~A13
- U6 pad 27: /Memory/~WR -> /~WR
- U6 pad 28: /Memory/+5V -> /+5V
- U6 pad 3: /Memory/A7 -> /~A7
- U6 pad 4: /Memory/A6 -> /~A6
- U6 pad 5: /Memory/A5 -> /~A5
- U6 pad 6: /Memory/A4 -> /~A4
- U6 pad 7: /Memory/A3 -> /~A3
- U6 pad 8: /Memory/A2 -> /~A2
- U6 pad 9: /Memory/A1 -> /~A1
- U7 pad 1: /Memory/A14 -> /~A14
- U7 pad 10: /Memory/A0 -> /~A0
- U7 pad 11: /Memory/D0 -> /~D0
- U7 pad 12: /Memory/D1 -> /~D1
- U7 pad 13: /Memory/D2 -> /~D2
- U7 pad 14: /Memory/GND -> /GND
- U7 pad 15: /Memory/D3 -> /~D3
- U7 pad 16: /Memory/D4 -> /~D4
- U7 pad 17: /Memory/D5 -> /~D5
- U7 pad 18: /Memory/D6 -> /~D6
- U7 pad 19: /Memory/D7 -> /~D7
- U7 pad 2: /Memory/A12 -> /~A12
- U7 pad 21: /Memory/A10 -> /~A10
- U7 pad 22: /Memory/~RD -> /~RD
- U7 pad 23: /Memory/A11 -> /~A11
- U7 pad 24: /Memory/A9 -> /~A9
- U7 pad 25: /Memory/A8 -> /~A8
- U7 pad 26: /Memory/A13 -> /~A13
- U7 pad 27: /Memory/~WR -> /~WR
- U7 pad 28: /Memory/+5V -> /+5V
- U7 pad 3: /Memory/A7 -> /~A7
- U7 pad 4: /Memory/A6 -> /~A6
- U7 pad 5: /Memory/A5 -> /~A5
- U7 pad 6: /Memory/A4 -> /~A4
- U7 pad 7: /Memory/A3 -> /~A3
- U7 pad 8: /Memory/A2 -> /~A2
- U7 pad 9: /Memory/A1 -> /~A1
- U9 pad 1: /ATA.sch/RESET -> Net-(Q2-Pad1)
- U9 pad 10: /CPU/RESET -> Net-(U9-Pad10)
- U9 pad 11: ~RESET -> /~D3
- U9 pad 12: (no net) -> Net-(U9-Pad12)
- U9 pad 13: (no net) -> /~D2
- U9 pad 2: Net-(U10-Pad1) -> /GND
- U9 pad 3: /CPU/~IORQ -> /~D7
- U9 pad 5: Net-(C2-Pad1) -> /~D6
- U9 pad 6: Net-(R11-Pad2) -> Net-(U9-Pad6)
- U9 pad 7: Net-(U9-Pad7) -> /~D5
- U9 pad 9: Net-(R11-Pad2) -> /~D4
- Y2 pad 1: Net-(C6-Pad1) -> Net-(C4-Pad1)
- Y2 pad 2: Net-(C5-Pad1) -> Net-(C3-Pad1)

Commit message: 1
Routing:
- net /+5V: track 0.00 -> 506.3 mm, vias 0 -> 2
- net /GND: track 0.00 -> 502.7 mm, vias 0 -> 1
- net /~A0: track 0.00 -> 214.9 mm, vias 0 -> 1
- net /~D2: track 0.00 -> 214.0 mm, vias 0 -> 2
- net /~D0: track 0.00 -> 204.2 mm
- net /~D4: track 0.00 -> 203.5 mm
- net /~WR: track 0.00 -> 197.2 mm, vias 0 -> 1
- net /~D7: track 0.00 -> 194.2 mm
- net /~D6: track 0.00 -> 189.5 mm, vias 0 -> 1
- net /~A15: track 0.00 -> 187.3 mm, vias 0 -> 3
- net /~D3: track 0.00 -> 176.7 mm, vias 0 -> 1
- net /~D1: track 0.00 -> 175.3 mm, vias 0 -> 1
- net /~D5: track 0.00 -> 174.7 mm, vias 0 -> 1
- net /~A1: track 0.00 -> 173.7 mm, vias 0 -> 3
- net /~A2: track 0.00 -> 169.0 mm
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
Commit message: 1
Parts:
- added C10: 1uf, Capacitor_SMD:C_0805_2012Metric, F.Cu at (61.1, 59.7)
- added C11: C, Capacitor_SMD:C_0805_2012Metric, F.Cu at (95.1, 33.0)
- added C12: 1uf, Capacitor_SMD:C_0805_2012Metric, F.Cu at (83.2, 59.9)
- added C13: 1uf, Capacitor_SMD:C_0805_2012Metric, F.Cu at (67.6, 34.0)
- added C14: 1uf, Capacitor_SMD:C_0805_2012Metric, F.Cu at (64.2, 42.6)
- added C15: 1uf, Capacitor_SMD:C_0805_2012Metric, F.Cu at (93.6, 105.8)
- added C16: 1uf, Capacitor_SMD:C_0805_2012Metric, F.Cu at (111.7, 51.7)
- added C17: 1uf, Capacitor_SMD:C_0805_2012Metric, F.Cu at (79.4, 51.3)
- added C18: 1uf, Capacitor_SMD:C_0805_2012Metric, F.Cu at (35.2, 43.5)
- added C19: 1uf, Capacitor_SMD:C_0805_2012Metric, F.Cu at (93.0, 38.1)
- added C20: 1uf, Capacitor_SMD:C_0805_2012Metric, F.Cu at (79.5, 48.9)
- added C21: CP1, Capacitor_THT:CP_Radial_D7.5mm_P2.50mm, F.Cu at (96.0, 112.1)
- added C22: 1uf, Capacitor_SMD:C_0805_2012Metric, F.Cu at (86.4, 32.1)
- added C5: 1uf, Capacitor_SMD:C_0805_2012Metric, F.Cu at (24.6, 73.3)
- added C6: 1uf, Capacitor_SMD:C_0805_2012Metric, F.Cu at (69.1, 114.8)
- added C7: 1uf, Capacitor_SMD:C_0805_2012Metric, F.Cu at (75.2, 100.6)
- added C8: 1uf, Capacitor_SMD:C_0805_2012Metric, F.Cu at (57.9, 101.5)
- added C9: 1uf, Capacitor_SMD:C_0805_2012Metric, F.Cu at (71.2, 106.7)
- added J3: PSX_JOYPAD_1, Connector_PinSocket_2.54mm:PinSocket_1x09_P2.54mm_Vertical, F.Cu at (17.1, 87.4)
- added J4: PSX_JOYPAD_2, Connector_PinSocket_2.54mm:PinSocket_1x09_P2.54mm_Vertical, F.Cu at (17.1, 61.8)
- added R12: 2k, Resistor_SMD:R_0805_2012Metric, F.Cu at (32.1, 28.4)
- added R16: 2k, Resistor_SMD:R_0805_2012Metric, F.Cu at (29.6, 28.4)
- added R4: 120, Resistor_SMD:R_0805_2012Metric, F.Cu at (34.7, 23.3)
- added R5: 120, Resistor_SMD:R_0805_2012Metric, F.Cu at (32.1, 23.3)
- added R6: 120, Resistor_SMD:R_0805_2012Metric, F.Cu at (37.2, 23.3)
- added R7: 120, Resistor_SMD:R_0805_2012Metric, F.Cu at (29.7, 23.3)
- added R8: 2k, Resistor_SMD:R_0805_2012Metric, F.Cu at (34.7, 28.4)
- added R9: 2k, Resistor_SMD:R_0805_2012Metric, F.Cu at (37.2, 28.4)
- added SW2: SW_DPDT_x2, Package_DIP:DIP-6_W7.62mm, F.Cu at (105.6, 26.6)
- added U3: PS2_DUAL, Connector_PinSocket_2.54mm:PS2DUAL, F.Cu at (78.8, 23.2)
- U13: value STC89C52-Vintage -> 89C51
- U6, U7: footprint Package_DIP:DIP-32_W15.24mm_Socket -> Package_DIP:DIP-28_W15.24mm_Socket
- moved R25 483.9 mm to (102.2, 51.8)
- moved U11 471.0 mm to (78.4, 54.1)
- moved R3 459.5 mm to (91.8, 32.0), turned to 90 degrees
- moved U5 459.1 mm to (70.2, 112.3), turned to 90 degrees
- moved D1 456.5 mm to (89.6, 28.2), turned to 90 degrees
- moved R1 454.8 mm to (91.8, 28.3), turned to 90 degrees
- moved R2 452.6 mm to (89.6, 32.0), turned to 90 degrees
- moved SW1 446.5 mm to (89.3, 24.4), turned to 90 degrees
- moved J1 444.4 mm to (109.1, 21.2), turned to 180 degrees
- moved JP1 437.7 mm to (40.4, 95.1), turned to 180 degrees
- moved JP2 436.9 mm to (40.4, 92.6), turned to 180 degrees
- moved Q1 433.4 mm to (83.8, 31.0), turned to 180 degrees
- moved U18 433.4 mm to (97.4, 54.1)
- moved U12 433.3 mm to (97.3, 43.1)
- moved U21 433.3 mm to (78.5, 43.1)
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Connections:
- C1 pad 1: /+5V -> Net-(C1-Pad1)
- J1 pad 1: /+5V -> Net-(C1-Pad1)
- J2 pad 39: Net-(J2-Pad39) -> /RESET
- U1 pad 1: Net-(U1-Pad1) -> PSX_CMD
- U1 pad 18: Net-(U1-Pad18) -> ~PSX_ACK
- U1 pad 19: Net-(U1-Pad19) -> PSX_DAT
- U1 pad 2: Net-(U1-Pad2) -> PSX_CLK
- U1 pad 3: Net-(U1-Pad3) -> ~PSX_SEL_1
- U1 pad 4: Net-(U1-Pad4) -> ~PSX_SEL_0
- U12 pad 13: Net-(U12-Pad13) -> ~RESET
- U13 pad 12: Net-(U13-Pad12) -> MOUSE_CLK
- U13 pad 13: Net-(U13-Pad13) -> KEYBOARD_CLK
- U13 pad 14: Net-(U13-Pad14) -> KEYBOARD_DAT
- U13 pad 15: Net-(U13-Pad15) -> MOUSE_DAT
Routing:
- net /GND: track 502.7 -> 665.7 mm
- net /RESET: track 110.0 -> 243.8 mm, vias 1 -> 0
- net Net-(Q2-Pad2): track 74.8 -> 6.79 mm, vias 1 -> 0
- net PSX_CMD: track 0.00 -> 64.9 mm
- net Net-(D10-Pad1): track 10.8 -> 70.6 mm, vias 0 -> 1
- net ~PSX_ACK: track 0.00 -> 57.3 mm
- net /+5V: track 506.3 -> 557.0 mm, vias 2 -> 3
- net Net-(R7-Pad1): track 0.00 -> 49.6 mm
- net PSX_CLK: track 0.00 -> 49.2 mm
- net PSX_DAT: track 0.00 -> 48.6 mm
- net /~D6: track 189.5 -> 237.2 mm, vias 1 -> 7
- net Net-(R5-Pad1): track 0.00 -> 43.0 mm, vias 0 -> 1
- net /~D1: track 175.3 -> 217.4 mm, vias 1 -> 3
- net /~D5: track 174.7 -> 214.9 mm, vias 1 -> 5
- net Net-(R4-Pad1): track 0.00 -> 39.6 mm
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- added copper zone on B.Cu, net (none)
- added copper zone on F.Cu, net (none)
- added copper zone on B.Cu, net /GND
- added copper zone on F.Cu, net /GND
Other:
- net class POWER added: clearance 0.2, trace_width 0.4, via_dia 0.8, via_drill 0.4

Commit message: 1
Parts:
- U13: value 89C51 -> STC89C52-Vintage
Connections:
- R11 pad 2: ~ENTER_ISP -> ~EXIT_BOOT
- U10 pad 15: ~ENTER_ISP -> ~EXIT_BOOT
- U12 pad 1: ~ENTER_ISP -> ~EXIT_BOOT
Routing:
- net ~EXIT_BOOT: track 0.00 -> 28.8 mm, vias 0 -> 2
- net ~ENTER_ISP: track 46.1 -> 36.5 mm, vias 1 -> 2
- net ~ISP: track 75.0 -> 77.4 mm
- net ~BOOTING: track 48.8 -> 50.9 mm
- net ISP: track 23.4 -> 24.2 mm
- net ~WR_BIOS: track 56.3 -> 57.1 mm
- net /~RD: track 171.4 -> 172.2 mm
- net Net-(Q2-Pad1): track 75.7 -> 76.3 mm
- net /GND: track 665.7 -> 666.3 mm
- net /~WR: track 219.1 -> 219.6 mm
- net ~RESET: track 85.7 -> 86.3 mm
- removed copper zone on B.Cu, net (none)
- removed copper zone on F.Cu, net (none)
- removed copper zone on B.Cu, net /GND
- removed copper zone on F.Cu, net /GND
